Commit message: Robust Transformation

File: src/vbm_project/vbm_project_env/urdf/camera.urdf (robot description, URDF)
Before this commit: robot camera, 4 links, 3 joints
Joints:
- joint world_to_base: origin (none) -> xyz=0 0 1.5 rpy=0 1.57 0

Commit message: Clustering and Transforms

File: src/vbm_project/vbm_project_env/urdf/camera.urdf (robot description, URDF)
Before this commit: robot camera, 4 links, 3 joints
Joints:
- joint world_to_base: origin xyz=0 0 1.5 rpy=0 1.57 0 -> xyz=0.4 0 1.5 rpy=0 2.0944 0
